File: hw/move-chirper/move-chirper.kicad_pcb (KiCad board)
At the start: 2 copper layers, 63.5 x 27.9 mm, 32 parts, among them J1 PIR, J2 piezo, J3 power in, J4 ISP reset, J5 ISP prog, J6 leds, J7 IR receiver blue-cyan, Q1 1N3904, Q2 BC546, Q3 BC546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

Commit message: hw update
Parts:
- added C7: 100n, Capacitor_THT:C_Disc_D5.0mm_W2.5mm_P2.50mm, F.Cu at (149.9, 55.9)
- added R10: 91k, Resistor_THT:R_Axial_DIN0207_L6.3mm_D2.5mm_P10.16mm_Horizontal, F.Cu at (154.9, 68.6)
- added R11: 4k7, Resistor_THT:R_Axial_DIN0207_L6.3mm_D2.5mm_P10.16mm_Horizontal, F.Cu at (160.0, 58.4)
- U2: value AMS1117-5.0 -> L78L05_TO92; footprint Package_TO_SOT_THT:TO-92L_Inline_Wide -> Package_TO_SOT_THT:TO-92_Inline_Wide
Connections:
- R2 pad 2: Net-(Q1-B) -> Net-(C7-Pad1)
- U2 pad 1: /gnd -> /+5
- U2 pad 2: /+5 -> /gnd
Routing:
- net Net-(C7-Pad1): track 0.00 -> 10.2 mm
- net Net-(Q1-B): track 17.0 -> 25.0 mm
- net /+12: track 107.3 -> 109.8 mm
- net /+5: track 69.3 -> 67.6 mm
- net /gnd: track 169.8 -> 171.0 mm
