File: hw/move-chirper/move-chirper.kicad_sch (KiCad schematic)
At the start: 26 parts, among them J1 PIR, J2 piezo, J3 Conn_01x03, J4 ISP reset, J5 ISP prog, J6 Conn_01x03, Q1 1N3904, Q2 NPN, Q3 NPN, Q4 NPN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

Commit message: wip: casing created all modules
Parts:
- removed U2: AMS1117-5.0, Package_TO_SOT_SMD:SOT-223-3_TabPin2, symbol Regulator_Linear:AMS1117-5.0
- added C5, C6: 100n, Capacitor_THT:C_Disc_D5.0mm_W2.5mm_P2.50mm, symbol Device:C
- added D2: D, Diode_THT:D_A-405_P10.16mm_Horizontal, symbol Device:D
- added J7: IR receiver blue-cyan, Connector_PinHeader_2.54mm:PinHeader_1x03_P2.54mm_Vertical, symbol Connector_Generic:Conn_01x03
- added Q5: 2N3904, Package_TO_SOT_THT:TO-92L_Inline_Wide, symbol Simulation_SPICE:NPN
- added R9: 1k, Resistor_THT:R_Axial_DIN0207_L6.3mm_D2.5mm_P10.16mm_Horizontal, symbol Device:R
- added U2: L78L05_TO92, Package_TO_SOT_THT:TO-92_Inline, symbol Regulator_Linear:L78L05_TO92
- C1, C2: footprint (none) -> Capacitor_THT:C_Disc_D5.0mm_W2.5mm_P2.50mm
- C3: footprint (none) -> Capacitor_THT:CP_Radial_D4.0mm_P2.00mm
- C4: footprint (none) -> Capacitor_THT:CP_Radial_D6.3mm_P2.50mm
- D1: value D -> shottky; footprint (none) -> Diode_THT:D_A-405_P10.16mm_Horizontal
- J1, J5: footprint (none) -> Connector_PinHeader_2.54mm:PinHeader_1x03_P2.54mm_Vertical
- J2, J4: footprint (none) -> Connector_PinHeader_2.54mm:PinHeader_1x02_P2.54mm_Vertical
- J3: value Conn_01x03 -> power in; footprint (none) -> Connector_PinHeader_2.54mm:PinHeader_1x03_P2.54mm_Vertical
- J6: value Conn_01x03 -> leds; footprint (none) -> Connector_PinHeader_2.54mm:PinHeader_1x04_P2.54mm_Vertical; symbol Connector_Generic:Conn_01x03 -> Connector_Generic:Conn_01x04
- L1: footprint (none) -> Inductor_THT:L_Radial_D10.5mm_P5.00mm_Abacron_AISR-01
- Q1: footprint (none) -> Package_TO_SOT_THT:TO-92L_Inline_Wide
- Q2, Q3, Q4: value NPN -> BC546; footprint (none) -> Package_TO_SOT_THT:TO-92L_Inline_Wide
- R1: footprint (none) -> Resistor_THT:R_Axial_DIN0309_L9.0mm_D3.2mm_P15.24mm_Horizontal
- R2, R3, R4, R5, R6, R7, R8: footprint (none) -> Resistor_THT:R_Axial_DIN0207_L6.3mm_D2.5mm_P10.16mm_Horizontal
- U1: footprint Package_SO:SOIC-8_3.9x4.9mm_P1.27mm -> Package_DIP:DIP-8_W7.62mm
Connections:
- net +12: now also J6.4 (Pin_4), D2.1 (K), U2.3 (VI)
- net +5: now also C5.2, C6.1, J7.2 (Pin_2), R9.1, U2.1 (VO)
- net gnd: now also C5.1, C6.2, D2.2 (A), J7.1 (Pin_1), Q5.3 (E), U2.2 (GND)
- net led3 renamed ir
- net ir: now also Q5.1 (C), R9.2
- new net: J7.3 (Pin_3), Q5.2 (B)

Commit message: hw update
Parts:
- added C7: 100n, Capacitor_THT:C_Disc_D5.0mm_W2.5mm_P2.50mm, symbol Device:C
- added R10: 91k, Resistor_THT:R_Axial_DIN0207_L6.3mm_D2.5mm_P10.16mm_Horizontal, symbol Device:R
- added R11: 4k7, Resistor_THT:R_Axial_DIN0207_L6.3mm_D2.5mm_P10.16mm_Horizontal, symbol Device:R
- U2: footprint Package_TO_SOT_THT:TO-92_Inline -> Package_TO_SOT_THT:TO-92_Inline_Wide
Connections:
- net +12: now also R10.1
- net gnd: now also R11.2
- net at Q1.2 (B): now also C7.2, R10.2, R11.1; no longer R2.2
- new net: C7.1, R2.2
Other:
- moved on the sheet: R2
Changed lines of the file:
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@@
 (kicad_sch (version 20230121) (generator eeschema)
   (paper "A4")
+  (title_block
+    (date "2025-09-19")
+  )
   (junction (at 234.95 74.93) (diameter 0) (color 0 0 0 0)
   )
@@
   (junction (at 43.18 85.09) (diameter 0) (color 0 0 0 0)
   )
+  (junction (at 226.06 91.44) (diameter 0) (color 0 0 0 0)
+  )
   (junction (at 234.95 62.23) (diameter 0) (color 0 0 0 0)
   )
@@
   (junction (at 54.61 72.39) (diameter 0) (color 0 0 0 0)
   )
+  (junction (at 229.87 62.23) (diameter 0) (color 0 0 0 0)
+  )
+  (wire (pts (xy 229.87 62.23) (xy 234.95 62.23))
+    (stroke (width 0) (type default))
+  )
   (wire (pts (xy 234.95 62.23) (xy 248.92 62.23))
     (stroke (width 0) (type default))
@@
     (stroke (width 0) (type default))
   )
+  (wire (pts (xy 226.06 78.74) (xy 226.06 74.93))
+    (stroke (width 0) (type default))
+  )
   (wire (pts (xy 143.51 91.44) (xy 127 91.44))
     (stroke (width 0) (type default))
   )
+  (wire (pts (xy 210.82 91.44) (xy 212.09 91.44))
+    (stroke (width 0) (type default))
+  )
   (wire (pts (xy 147.32 80.01) (xy 144.78 80.01))
     (stroke (width 0) (type default))
   )
+  (wire (pts (xy 229.87 74.93) (xy 229.87 62.23))
+    (stroke (width 0) (type default))
+  )
   (wire (pts (xy 43.18 132.08) (xy 50.8 132.08))
     (stroke (width 0) (type default))
@@
     (stroke (width 0) (type default))
   )
+  (wire (pts (xy 226.06 91.44) (xy 226.06 96.52))
+    (stroke (width 0) (type default))
+  )
+  (wire (pts (xy 31.75 157.48) (xy 31.75 139.7))
+    (stroke (width 0) (type default))
+  )
+  (wire (pts (xy 24.13 149.86) (xy 24.13 142.24))
+    (stroke (width 0) (type default))
+  )
+  (wire (pts (xy 31.75 72.39) (xy 31.75 73.66))
+    (stroke (width 0) (type default))
+  )
+  (wire (pts (xy 248.92 62.23) (xy 248.92 67.31))
+    (stroke (width 0) (type default))
+  )
+  (wire (pts (xy 234.95 83.82) (xy 234.95 86.36))
+    (stroke (width 0) (type default))
+  )
+  (wire (pts (xy 106.68 19.05) (xy 129.54 19.05))
+    (stroke (width 0) (type default))
+  )
+  (wire (pts (xy 43.18 85.09) (xy 54.61 85.09))
+    (stroke (width 0) (type default))
+  )
+  (wire (pts (xy 144.78 39.37) (xy 154.94 39.37))
+    (stroke (width 0) (type default))
+  )
+  (wire (pts (xy 223.52 64.77) (xy 223.52 62.23))
+    (stroke (width 0) (type default))
+  )
+  (wire (pts (xy 20.32 157.48) (xy 31.75 157.48))
+    (stroke (width 0) (type default))
+  )
+  (wire (pts (xy 50.8 72.39) (xy 54.61 72.39))
+    (stroke (width 0) (type default))
+  )
+  (wire (pts (xy 144.78 31.75) (xy 154.94 31.75))
+    (stroke (width 0) (type default))
+  )
+  (wire (pts (xy 43.18 85.09) (xy 43.18 80.01))
+    (stroke (width 0) (type default))
+  )
+  (wire (pts (xy 219.71 91.44) (xy 226.06 91.44))
+    (stroke (width 0) (type default))
+  )
+  (wire (pts (xy 226.06 74.93) (xy 229.87 74.93))
+    (stroke (width 0) (type default))
+  )
   (wire (pts (xy 226.06 91.44) (xy 227.33 91.44))
     (stroke (width 0) (type default))
   )
-  (wire (pts (xy 31.75 157.48) (xy 31.75 139.7))
-    (stroke (width 0) (type default))
-  )
-  (wire (pts (xy 24.13 149.86) (xy 24.13 142.24))
-    (stroke (width 0) (type default))
-  )
-  (wire (pts (xy 31.75 72.39) (xy 31.75 73.66))
-    (stroke (width 0) (type default))
-  )
-  (wire (pts (xy 248.92 62.23) (xy 248.92 67.31))
-    (stroke (width 0) (type default))
-  )
-  (wire (pts (xy 234.95 83.82) (xy 234.95 86.36))
-    (stroke (width 0) (type default))
-  )
-  (wire (pts (xy 106.68 19.05) (xy 129.54 19.05))
-    (stroke (width 0) (type default))
-  )
-  (wire (pts (xy 43.18 85.09) (xy 54.61 85.09))
-    (stroke (width 0) (type default))
-  )
-  (wire (pts (xy 144.78 39.37) (xy 154.94 39.37))
-    (stroke (width 0) (type default))
-  )
-  (wire (pts (xy 223.52 64.77) (xy 223.52 62.23))
-    (stroke (width 0) (type default))
-  )
-  (wire (pts (xy 20.32 157.48) (xy 31.75 157.48))
-    (stroke (width 0) (type default))
-  )
-  (wire (pts (xy 50.8 72.39) (xy 54.61 72.39))
-    (stroke (width 0) (type default))
-  )
-  (wire (pts (xy 144.78 31.75) (xy 154.94 31.75))
-    (stroke (width 0) (type default))
-  )
-  (wire (pts (xy 43.18 85.09) (xy 43.18 80.01))
-    (stroke (width 0) (type default))
-  )
   (wire (pts (xy 234.95 74.93) (xy 234.95 76.2))
     (stroke (width 0) (type default))
@@
     (stroke (width 0) (type default))
   )
+  (wire (pts (xy 226.06 104.14) (xy 226.06 106.68))
+    (stroke (width 0) (type default))
+  )
+  (wire (pts (xy 226.06 106.68) (xy 234.95 106.68))
+    (stroke (width 0) (type default))
+  )
+  (wire (pts (xy 226.06 86.36) (xy 226.06 91.44))
+    (stroke (width 0) (type default))
+  )
   (wire (pts (xy 24.13 21.59) (xy 31.75 21.59))
     (stroke (width 0) (type default))
@@
     (stroke (width 0) (type default))
   )
-  (wire (pts (xy 223.52 62.23) (xy 234.95 62.23))
+  (wire (pts (xy 223.52 62.23) (xy 229.87 62.23))
     (stroke (width 0) (type default))
   )
@@
     (effects (font (size 1.27 1.27)) (justify left bottom))
   )
-  (label "piezo" (at 218.44 91.44 180) (fields_autoplaced)
+  (label "piezo" (at 203.2 91.44 180) (fields_autoplaced)
     (effects (font (size 1.27 1.27)) (justify right bottom))
   )
@@
       (effects (font (size 1.27 1.27)))
     )
-    (property "Footprint" "Package_TO_SOT_THT:TO-92_Inline" (at 43.18 66.675 0)
+    (property "Footprint" "Package_TO_SOT_THT:TO-92_Inline_Wide" (at 43.18 66.675 0)
       (effects (font (size 1.27 1.27) italic) hide)
     )
@@
     )
   )
+  (symbol (lib_id "Device:R") (at 226.06 82.55 0) (unit 1)
+    (in_bom yes) (on_board yes) (dnp no) (fields_autoplaced)
+    (property "Reference" "R10" (at 228.6 81.28 0)
+      (effects (font (size 1.27 1.27)) (justify left))
+    )
+    (property "Value" "91k" (at 228.6 83.82 0)
+      (effects (font (size 1.27 1.27)) (justify left))
+    )
+    (property "Footprint" "Resistor_THT:R_Axial_DIN0207_L6.3mm_D2.5mm_P10.16mm_Horizontal" (at 224.282 82.55 90)
+      (effects (font (size 1.27 1.27)) hide)
+    )
+    (property "Datasheet" "~" (at 226.06 82.55 0)
+      (effects (font (size 1.27 1.27)) hide)
+    )
+    (pin "2")
+    (pin "1")
+    (instances
+      (project "move-chirper"
+        (path "/48a3b2a7-7358-4dc7-bf03-812c34765dda"
+          (reference "R10") (unit 1)
+        )
+      )
+    )
+  )
   (symbol (lib_id "Device:C_Polarized") (at 19.05 77.47 0) (unit 1)
     (in_bom yes) (on_board yes) (dnp no) (fields_autoplaced)
@@
     )
   )
+  (symbol (lib_id "Device:R") (at 226.06 100.33 0) (unit 1)
+    (in_bom yes) (on_board yes) (dnp no) (fields_autoplaced)
+    (property "Reference" "R11" (at 228.6 99.06 0)
+      (effects (font (size 1.27 1.27)) (justify left))
+    )
+    (property "Value" "4k7" (at 228.6 101.6 0)
+      (effects (font (size 1.27 1.27)) (justify left))
+    )
+    (property "Footprint" "Resistor_THT:R_Axial_DIN0207_L6.3mm_D2.5mm_P10.16mm_Horizontal" (at 224.282 100.33 90)
+      (effects (font (size 1.27 1.27)) hide)
+    )
+    (property "Datasheet" "~" (at 226.06 100.33 0)
+      (effects (font (size 1.27 1.27)) hide)
+    )
+    (pin "1")
+    (pin "2")
+    (instances
+      (project "move-chirper"
+        (path "/48a3b2a7-7358-4dc7-bf03-812c34765dda"
+          (reference "R11") (unit 1)
+        )
+      )
+    )
+  )
   (symbol (lib_id "Device:C") (at 54.61 77.47 0) (unit 1)
     (in_bom yes) (on_board yes) (dnp no) (fields_autoplaced)
@@
     )
   )
-  (symbol (lib_id "Device:R") (at 222.25 91.44 90) (unit 1)
-    (in_bom yes) (on_board yes) (dnp no) (fields_autoplaced)
-    (property "Reference" "R2" (at 222.25 85.09 90)
-      (effects (font (size 1.27 1.27)))
-    )
-    (property "Value" "2k" (at 222.25 87.63 90)
-      (effects (font (size 1.27 1.27)))
-    )
-    (property "Footprint" "Resistor_THT:R_Axial_DIN0207_L6.3mm_D2.5mm_P10.16mm_Horizontal" (at 222.25 93.218 90)
-      (effects (font (size 1.27 1.27)) hide)
-    )
-    (property "Datasheet" "~" (at 222.25 91.44 0)
+  (symbol (lib_id "Device:R") (at 207.01 91.44 90) (unit 1)
+    (in_bom yes) (on_board yes) (dnp no) (fields_autoplaced)
+    (property "Reference" "R2" (at 207.01 85.09 90)
+      (effects (font (size 1.27 1.27)))
+    )
+    (property "Value" "2k" (at 207.01 87.63 90)
+      (effects (font (size 1.27 1.27)))
+    )
+    (property "Footprint" "Resistor_THT:R_Axial_DIN0207_L6.3mm_D2.5mm_P10.16mm_Horizontal" (at 207.01 93.218 90)
+      (effects (font (size 1.27 1.27)) hide)
+    )
+    (property "Datasheet" "~" (at 207.01 91.44 0)
       (effects (font (size 1.27 1.27)) hide)
     )
@@
         )
       )
+    )
+  )
+  (symbol (lib_id "Device:C") (at 215.9 91.44 90) (unit 1)
+    (in_bom yes) (on_board yes) (dnp no) (fields_autoplaced)
+    (property "Reference" "C7" (at 215.9 83.82 90)
+      (effects (font (size 1.27 1.27)))
+    )
+    (property "Value" "100n" (at 215.9 86.36 90)
+      (effects (font (size 1.27 1.27)))
+    )
+    (property "Footprint" "Capacitor_THT:C_Disc_D5.0mm_W2.5mm_P2.50mm" (at 219.71 90.4748 0)
+      (effects (font (size 1.27 1.27)) hide)
+    )
+    (property "Datasheet" "~" (at 215.9 91.44 0)
+      (effects (font (size 1.27 1.27)) hide)
+    )
+    (pin "1")
+    (pin "2")
+    (instances
+      (project "move-chirper"
+        (path "/48a3b2a7-7358-4dc7-bf03-812c34765dda"
+          (reference "C7") (unit 1)
+        )
+      )
